File: PCB/V2.1 KiCad Version/ResQ KiCad Version/ResQ KiCad Version.kicad_pcb (KiCad board)
At the start: 2 copper layers, 7 parts, among them J1 Spare 1, J2 Spare 2, J3 OLED, J4 SD Card, J5 GPS, U1 WeMos_D1_mini

Commit message: oled pinout reversal
Connections:
- J3 pad 1: 3V3 -> GND
- J3 pad 2: GND -> 3V3

Commit message: Scematic fixes
Parts:
- removed BT1: 5V, Connector_PinSocket_2.54mm:PinSocket_1x02_P2.54mm_Vertical
- added B1: 5V, Connector_PinSocket_2.54mm:PinSocket_1x02_P2.54mm_Vertical, F.Cu at (212.1, 116.8)
- added J6: Radio, Connector_PinSocket_2.54mm:PinSocket_1x04_P2.54mm_Vertical, F.Cu at (163.8, 108.0)
- added R1: 10k, Resistor_SMD:R_0201_0603Metric, F.Cu at (180.1, 103.2)
- moved J1 10.9 mm to (181.6, 148.6)
- moved J2 10.9 mm to (191.8, 148.6)
Connections:
- U1 pad 1: Net-(U1-Pad1) -> (no net)
- U1 pad 15: Net-(U1-Pad15) -> RX
- U1 pad 16: Net-(U1-Pad16) -> TX

Commit message: Updates
Parts:
- moved J6 45.0 mm to (205.7, 124.5)
- moved J3 31.5 mm to (194.3, 132.1)
- moved R1 18.0 mm to (194.3, 114.3)
- moved B1 7.41 mm to (205.7, 113.0)
- moved J5 5.24 mm to (181.6, 132.1)

Commit message: Camera Module added
Parts:
- J2: value Spare 2 -> Cam

Commit message: Beginning PCB V2.Xxx Design
Parts:
- moved B1 42.6 mm to (172.5, 139.7)
- moved J6 33.3 mm to (172.5, 124.7)
- moved J3 30.9 mm to (172.2, 110.5)
- moved J1 13.2 mm to (187.2, 136.7)
- moved J2 11.9 mm to (191.8, 136.7)
- moved J5 7.47 mm to (180.3, 124.7)
Connections:
- J5 pad 1: GND -> 3V3
- J5 pad 2: D4 -> D3
- J5 pad 3: D3 -> D4
- J5 pad 4: 3V3 -> GND
- J6 pad 1: GND -> 3V3
- J6 pad 2: 3V3 -> GND
Other:
- board outline added: 31.5 x 36.1 mm

Commit message: PCB Version 2.1 routed
Parts:
- added REF**: OSHW-Logo_5.7x6mm_SilkScreen, Symbol:OSHW-Logo_5.7x6mm_SilkScreen, F.Cu at (187.2, 124.5)
- J1: value Spare 1 -> SP1
- R1: footprint Resistor_SMD:R_0201_0603Metric -> Resistor_SMD:R_0805_2012Metric_Pad1.15x1.40mm_HandSolder
- U1: value WeMos_D1_mini -> WeMos
- moved B1 26.7 mm to (199.1, 138.9)
- moved J6 24.0 mm to (194.6, 134.1)
- moved J2 20.2 mm to (172.5, 142.5), turned to 180 degrees
- moved J5 10.8 mm to (185.7, 134.1)
- moved J1 8.89 mm to (180.1, 142.0), turned to 180 degrees
- moved R1 1.80 mm to (195.6, 115.6), turned to 90 degrees
Routing:
- net 3V3: track 0.00 -> 97.3 mm
- net GND: track 0.00 -> 89.3 mm, vias 0 -> 4
- net MISO: track 0.00 -> 43.0 mm
- net SCL: track 0.00 -> 32.1 mm
- net SDA: track 0.00 -> 32.1 mm
- net MOSI: track 0.00 -> 30.6 mm
- net CLK: track 0.00 -> 28.8 mm
- net CS: track 0.00 -> 25.9 mm
- net A0: track 0.00 -> 24.4 mm
- net TX: track 0.00 -> 23.5 mm
- net RX: track 0.00 -> 23.5 mm
- net D4: track 0.00 -> 19.2 mm, vias 0 -> 1
- net D3: track 0.00 -> 18.5 mm, vias 0 -> 1
- net D0: track 0.00 -> 16.3 mm
- net 5V: track 0.00 -> 3.59 mm
- added copper zone on B.Cu, net GND
- added copper zone on F.Cu, net GND
Other:
- outline, holes or cut-outs redrawn
- board text added: "ResQ"
- board text added: "ResQ V2.1 www.mkme.org"

Commit message: PCB Updates
Parts:
- REF**: value OSHW-Logo_5.7x6mm_SilkScreen -> (none)
Other:
- board text added: "2020"
- board text added: "Eric @MKMEORG"
- board text removed: "ResQ"
